File: Hardware/KiCAD/Cobalt-Cowboy.kicad_pcb (KiCad board)
At the start: 2 copper layers, 138.1 x 102 mm, 154 parts, among them IC1 BQ24193RGER, IC3 ISL91127IRNZ-T7A, IC4 PCF8575PWR, IC5 SA630D_01,118, IC6 SA630D_01,118, J1 USB_C_Receptacle, J2 1x15, J3 1x15, J4 SD_Card, J5 Conn_Coaxial_UHF, J6 Peripherals, J8 Peripherals, SW1 SW_Push, SW10 *, SW11 4, SW12 5, SW13 6, SW14 0, SW15 7, SW16 8, SW17 9, SW18 #, SW19 PTT, SW2 SW_Push, SW3 MENU, SW4 UP, SW5 DOWN, SW6 EXIT, SW7 1, SW8 2, SW9 3, U2 ESP32-C3-WROOM-02, U3 CC1200RHBR, X1 40 MHz

Commit message: feat: Plot updated schematics #11
Parts:
- added IC8: GRF5504, Cobalt_Cowboy:QFN50P300X300X90-17N_GRF5504, F.Cu at (179.3, 70.2)
- added IC9: GRF5504, Cobalt_Cowboy:QFN50P300X300X90-17N_GRF5504, F.Cu at (179.3, 75.5)
- L1: footprint Inductor_SMD:L_0603_1608Metric -> Inductor_SMD:L_Coilcraft_XxL4020
- moved L1 0.76 mm to (125.2, 87.4)
- moved R34 0.24 mm to (128.9, 89.2)
- moved R25 0.23 mm to (128.9, 90.7)
Routing:
- net /Power_System/V_{SYS}: track 25.2 -> 23.7 mm
- net Net-(IC3-EN): track 17.4 -> 16.3 mm
